Commit message: added collision properties to the urdf

File: urdf/robot_arm_urdf_macro.xacro (robot description, xacro)
@@ -17,4 +17,10 @@
                 </material>
             </visual>
+            <collision>
+                <origin xyz="0.0075 -0.0685027 -0.2" rpy="0 -0 0" />
+                <geometry>
+                    <mesh filename="package://preentend_description/meshes/linear_axis_track_link.stl" scale="1 1 1" />
+                </geometry>
+            </collision>
         </link>
         <link name="${prefix}_linear_axis_carrier_link">
@@ -34,4 +40,10 @@
                 </material>
             </visual>
+            <collision>
+                <origin xyz="0.0075 -0.0685027 -0.2" rpy="0 -0 0" />
+                <geometry>
+                    <mesh filename="package://preentend_description/meshes/linear_axis_carrier_link.stl" scale="1 1 1" />
+                </geometry>
+            </collision>
         </link>
         <link name="${prefix}_base_link">
@@ -51,4 +63,10 @@
                 </material>
             </visual>
+            <collision>
+                <origin xyz="0.0075 -0.0685027 -0.2" rpy="0 -0 0" />
+                <geometry>
+                    <mesh filename="package://preentend_description/meshes/base_link.stl" scale="1 1 1" />
+                </geometry>
+            </collision>
         </link>
         <link name="${prefix}_link1">
@@ -68,4 +86,10 @@
                 </material>
             </visual>
+            <collision>
+                <origin xyz="0.0075 -0.0685027 -0.2" rpy="0 -0 0" />
+                <geometry>
+                    <mesh filename="package://preentend_description/meshes/link1.stl" scale="1 1 1" />
+                </geometry>
+            </collision>
         </link>
         <link name="${prefix}_link2">
@@ -85,4 +109,10 @@
                 </material>
             </visual>
+            <collision>
+                <origin xyz="0.0075 -0.0685027 -0.2" rpy="0 -0 0" />
+                <geometry>
+                    <mesh filename="package://preentend_description/meshes/link2.stl" scale="1 1 1" />
+                </geometry>
+            </collision>
         </link>
         <link name="${prefix}_link3">
@@ -102,4 +132,10 @@
                 </material>
             </visual>
+            <collision>
+                <origin xyz="0.0075 -0.0685027 -0.2" rpy="0 -0 0" />
+                <geometry>
+                    <mesh filename="package://preentend_description/meshes/link3.stl" scale="1 1 1" />
+                </geometry>
+            </collision>
         </link>
         <link name="${prefix}_link4">
@@ -119,4 +155,10 @@
                 </material>
             </visual>
+            <collision>
+                <origin xyz="0.0075 -0.0685027 -0.2" rpy="0 -0 0" />
+                <geometry>
+                    <mesh filename="package://preentend_description/meshes/link4.stl" scale="1 1 1" />
+                </geometry>
+            </collision>
         </link>
         <link name="${prefix}_link5">
@@ -136,4 +178,10 @@
                 </material>
             </visual>
+            <collision>
+                <origin xyz="0.0075 -0.0685027 -0.2" rpy="0 -0 0" />
+                <geometry>
+                    <mesh filename="package://preentend_description/meshes/link5.stl" scale="1 1 1" />
+                </geometry>
+            </collision>
         </link>
         <link name="${prefix}_flange_link">
@@ -152,4 +200,10 @@
                 </material>
             </visual>
+            <collision>
+                <origin xyz="0.0075 -0.0685027 -0.2" rpy="0 -0 0" />
+                <geometry>
+                    <mesh filename="package://preentend_description/meshes/flange_link.stl" scale="1 1 1" />
+                </geometry>
+            </collision>
         </link>
         <joint name="${prefix}_linear_axis_joint" type="prismatic">

Commit message: refactored collision origins in urdf

File: urdf/robot_arm_urdf_macro.xacro (robot description, xacro)
@@ -41,5 +41,5 @@
             </visual>
             <collision>
-                <origin xyz="0.0075 -0.0685027 -0.2" rpy="0 -0 0" />
+                <origin xyz="0.106514 -0.115615 -0.239552" rpy="0 -0 0" />
                 <geometry>
                     <mesh filename="package://preentend_description/meshes/linear_axis_carrier_link.stl" scale="1 1 1" />
@@ -64,5 +64,5 @@
             </visual>
             <collision>
-                <origin xyz="0.0075 -0.0685027 -0.2" rpy="0 -0 0" />
+                <origin xyz="0 0 0" rpy="0 -0 0" />
                 <geometry>
                     <mesh filename="package://preentend_description/meshes/base_link.stl" scale="1 1 1" />
@@ -87,5 +87,5 @@
             </visual>
             <collision>
-                <origin xyz="0.0075 -0.0685027 -0.2" rpy="0 -0 0" />
+                <origin xyz="-0.0589974 0.0447591 0.00389295" rpy="0 -0 0" />
                 <geometry>
                     <mesh filename="package://preentend_description/meshes/link1.stl" scale="1 1 1" />
@@ -110,5 +110,5 @@
             </visual>
             <collision>
-                <origin xyz="0.0075 -0.0685027 -0.2" rpy="0 -0 0" />
+                <origin xyz="-0.149564 0.0561702 0.00945553" rpy="0 -0 0" />
                 <geometry>
                     <mesh filename="package://preentend_description/meshes/link2.stl" scale="1 1 1" />
@@ -133,5 +133,5 @@
             </visual>
             <collision>
-                <origin xyz="0.0075 -0.0685027 -0.2" rpy="0 -0 0" />
+                <origin xyz="0.0543897 0.0843386 -0.0037732" rpy="0 -0 0" />
                 <geometry>
                     <mesh filename="package://preentend_description/meshes/link3.stl" scale="1 1 1" />
@@ -156,5 +156,5 @@
             </visual>
             <collision>
-                <origin xyz="0.0075 -0.0685027 -0.2" rpy="0 -0 0" />
+                <origin xyz="9.47542e-05 -1.5431e-05 0.109729" rpy="0 -0 0" />
                 <geometry>
                     <mesh filename="package://preentend_description/meshes/link4.stl" scale="1 1 1" />
@@ -179,5 +179,5 @@
             </visual>
             <collision>
-                <origin xyz="0.0075 -0.0685027 -0.2" rpy="0 -0 0" />
+                <origin xyz="0.043837 -0.100762 -6.06011e-18" rpy="0 -0 0" />
                 <geometry>
                     <mesh filename="package://preentend_description/meshes/link5.stl" scale="1 1 1" />
@@ -201,5 +201,5 @@
             </visual>
             <collision>
-                <origin xyz="0.0075 -0.0685027 -0.2" rpy="0 -0 0" />
+                <origin xyz="2.92246e-17 1.06541e-16 -0.0102682" rpy="0 -0 0" />
                 <geometry>
                     <mesh filename="package://preentend_description/meshes/flange_link.stl" scale="1 1 1" />
